File: Amplifier.kicad_sch (KiCad schematic)
At the start: 5 parts, among them U7 MAX98357A

Commit message: Recreated symbol/footprint libraries, added 3D models and Git LFS
Parts:
- removed U7: MAX98357A, symbol Custom_symbols:Adafruit_I2S_MAX98357A
- added U7: MAX98357A, symbol Project_symbols:Adafruit_I2S_MAX98357A
Connections:
- net BCLK: now also U7.2 (BCLK)
- net DIN: now also U7.3 (DIN)
- net GND: now also U7.6 (GND)
- net LRC: now also U7.1 (LRC)
- net VAMP: now also U7.7 (Vin)
- net at R27.2: now also U7.5 (SD)
- net at R24.2, R25.1: now also U7.4 (GAIN)
Changed lines of the file:
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@@
 	)
 	(symbol
-		(lib_id "Custom_symbols:Adafruit_I2S_MAX98357A")
+		(lib_id "Project_symbols:Adafruit_I2S_MAX98357A")
 		(at 138.43 86.36 0)
 		(unit 1)
@@
 			)
 		)
-		(pin "6"
+		(pin "1"
+		)
+		(pin "2"
 		)
 		(pin "4"
 		)
-		(pin "2"
+		(pin "5"
 		)
 		(pin "7"
@@
 		(pin "3"
 		)
-		(pin "5"
-		)
-		(pin "1"
+		(pin "6"
 		)
 		(instances
-			(project "StackLightDriver"
+			(project ""
 				(path "/d031313b-f769-488e-86bb-cea64c97ce3a/222c9d07-b657-4a9a-b551-efe9cdbeb418"
 					(reference "U7")

Commit message: Added models and footprint for Adafruit Max98357
Parts:
- U7: footprint (none) -> Project_footprints:Adafruit_I2S_MAX98357A
Changed lines of the file:
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@@
 			)
 		)
-		(property "Footprint" ""
+		(property "Footprint" "Project_footprints:Adafruit_I2S_MAX98357A"
 			(at 138.43 86.36 0)
 			(effects
